File: KiCad/Port_Starboard_ARM.kicad_sch (KiCad schematic)
At the start: 0 parts

Commit message: PS Arm PCB added
Parts:
- added J4: (no value), My_Library:Staggered_3_pin_conn, symbol My_Library:Staggered_3_pin_conn
- added L17, L18: (no value), My_Library:strip_WS2212, symbol My_Library:Strip_WS2212
Connections:
- new net: J4.1 (Gnd), L17.1 (Gnd), L18.1 (Gnd)
- new net: J4.2 (Dout), L17.2 (Din)
- new net: J4.3 (Vcc), L17.3 (Vcc), L18.3 (Vcc)
- new net: L17.5 (Dout), L18.2 (Din)
