File: KiCad/Tower Connector and PS Arm.kicad_pcb (KiCad board)
At the start: 2 copper layers, 74 x 12 mm, 3 parts, among them J1 Conn_01x03_Socket

Commit message: PS Arm PCB added
Parts:
- added J4: ~, My_Library:Staggered_3_pin_conn, F.Cu at (156.3, 57.4)
- added L1: ~, My_Library:strip_WS2212, F.Cu at (200.4, 62.5)
- added L2: ~, My_Library:strip_WS2212, F.Cu at (109.2, 67.6)
Routing:
- net Net-(L1-Dout): track 0.00 -> 94.2 mm, vias 0 -> 2
- net Net-(J4-Gnd): track 0.00 -> 83.3 mm, vias 0 -> 2
- net Net-(J4-Vcc): track 0.00 -> 83.2 mm
- net Net-(J4-Dout): track 0.00 -> 38.8 mm
Other:
- board size 74 x 12 mm -> 110 x 50 mm
